File: argon/argon.sch (KiCad schematic (older format))
At the start: 5 parts

Commit message: Add EEPROM & fix libs
Parts:
- added R? (x2): 10R, symbol Device:R
- added R?: 2.2K, symbol Device:R
- added R? (x3): 10K, symbol Device:R
- added U?: 93LCxxA, symbol ArgonComponents:93LCxxA
- J?: value USB_B_Micro_Alicja -> USB; symbol ConnectorA:USB_B_Micro_Alicja -> ArgonComponents:USB_B_Micro
Connections:
- net labels added: VCC
- wire segments 40 -> 66
Changed lines of the file:
@@
 Comment4 ""
 $EndDescr
-$Comp
-L ConnectorA:USB_B_Micro_Alicja J?
-U 1 1 5FCEC245
-P 2000 2550
-F 0 "J?" H 2053 3017 50  0000 C CNN
-F 1 "USB_B_Micro_Alicja" H 2053 2926 50  0000 C CNN
-F 2 "" H 2150 2400 50  0001 C CNN
-F 3 "~" H 2150 2400 50  0001 C CNN
-	1    2000 2550
-	1    0    0    -1
-$EndComp
-Wire Wire Line
-	4500 2550 2300 2550
-Wire Wire Line
-	2300 2650 4500 2650
-Wire Wire Line
-	1850 2950 1850 3500
-Wire Wire Line
-	1950 3500 1950 2950
-$Comp
-L power:GND #PWR?
-U 1 1 5FCEE675
-P 1900 3650
-F 0 "#PWR?" H 1900 3400 50  0001 C CNN
-F 1 "GND" H 1905 3477 50  0000 C CNN
-F 2 "" H 1900 3650 50  0001 C CNN
-F 3 "" H 1900 3650 50  0001 C CNN
-	1    1900 3650
-	1    0    0    -1
-$EndComp
-Wire Wire Line
-	1850 3500 1900 3500
-Wire Wire Line
-	1900 3650 1900 3500
-Connection ~ 1900 3500
-Wire Wire Line
-	1900 3500 1950 3500
+Wire Wire Line
+	4500 2550 4050 2550
+Wire Wire Line
+	2300 2650 3750 2650
 NoConn ~ 2300 2750
 $Comp
@@
 Wire Wire Line
 	5600 5850 5700 5850
+Wire Wire Line
+	3750 2550 2300 2550
+$Comp
+L Device:R R?
+U 1 1 5FD08DDB
+P 3900 2650
+F 0 "R?" V 3850 2450 50  0000 C CNN
+F 1 "10R" V 3850 2850 50  0000 C CNN
+F 2 "" V 3830 2650 50  0001 C CNN
+F 3 "~" H 3900 2650 50  0001 C CNN
+	1    3900 2650
+	0    1    1    0
+$EndComp
+Wire Wire Line
+	4050 2650 4500 2650
+$Comp
+L Device:R R?
+U 1 1 5FD08843
+P 3900 2550
+F 0 "R?" V 3850 2350 50  0000 C CNN
+F 1 "10R" V 3850 2750 50  0000 C CNN
+F 2 "" V 3830 2550 50  0001 C CNN
+F 3 "~" H 3900 2550 50  0001 C CNN
+	1    3900 2550
+	0    1    1    0
+$EndComp
+Wire Wire Line
+	1900 3050 1950 3050
+Connection ~ 1900 3050
+Wire Wire Line
+	1900 3200 1900 3050
+Wire Wire Line
+	1850 3050 1900 3050
+$Comp
+L power:GND #PWR?
+U 1 1 5FCEE675
+P 1900 3200
+F 0 "#PWR?" H 1900 2950 50  0001 C CNN
+F 1 "GND" H 1905 3027 50  0000 C CNN
+F 2 "" H 1900 3200 50  0001 C CNN
+F 3 "" H 1900 3200 50  0001 C CNN
+	1    1900 3200
+	1    0    0    -1
+$EndComp
+Wire Wire Line
+	1850 3050 1850 2950
+Wire Wire Line
+	1950 2950 1950 3050
+$Comp
+L power:GND #PWR?
+U 1 1 5FD16F0D
+P 1500 4350
+F 0 "#PWR?" H 1500 4100 50  0001 C CNN
+F 1 "GND" H 1505 4177 50  0000 C CNN
+F 2 "" H 1500 4350 50  0001 C CNN
+F 3 "" H 1500 4350 50  0001 C CNN
+	1    1500 4350
+	1    0    0    -1
+$EndComp
+Wire Wire Line
+	1800 4250 1500 4250
+Wire Wire Line
+	1500 4250 1500 4350
+$Comp
+L ArgonComponents:USB_B_Micro J?
+U 1 1 5FCEC245
+P 2000 2550
+F 0 "J?" H 2000 2900 50  0000 C CNN
+F 1 "USB" H 2200 2200 50  0000 R CNN
+F 2 "" H 2150 2400 50  0001 C CNN
+F 3 "~" H 2150 2400 50  0001 C CNN
+	1    2000 2550
+	1    0    0    -1
+$EndComp
+Text GLabel 1400 3650 0    50   Input ~ 0
+VCC
+Wire Wire Line
+	1500 4150 1800 4150
+Wire Wire Line
+	2500 4450 2550 4450
+Connection ~ 2550 4450
+Wire Wire Line
+	2550 4450 2800 4450
+Wire Wire Line
+	2500 4250 2950 4250
+Connection ~ 2950 4250
+Wire Wire Line
+	2950 4250 4500 4250
+Wire Wire Line
+	2500 4150 3350 4150
+Connection ~ 3350 4150
+Wire Wire Line
+	3350 4150 4500 4150
+Wire Wire Line
+	2950 3700 2950 3650
+$Comp
+L Device:R R?
+U 1 1 5FD48574
+P 2950 3850
+F 0 "R?" H 2850 3850 50  0000 C CNN
+F 1 "10K" V 3050 3850 50  0000 C CNN
+F 2 "" V 2880 3850 50  0001 C CNN
+F 3 "~" H 2950 3850 50  0001 C CNN
+	1    2950 3850
+	-1   0    0    1
+$EndComp
+$Comp
+L Device:R R?
+U 1 1 5FD47A57
+P 2550 3850
+F 0 "R?" H 2450 3850 50  0000 C CNN
+F 1 "10K" V 2650 3850 50  0000 C CNN
+F 2 "" V 2480 3850 50  0001 C CNN
+F 3 "~" H 2550 3850 50  0001 C CNN
+	1    2550 3850
+	-1   0    0    1
+$EndComp
+Wire Wire Line
+	2950 3650 3350 3650
+Wire Wire Line
+	3350 3650 3350 3700
+Connection ~ 2950 3650
+Wire Wire Line
+	2550 3650 2550 3700
+Wire Wire Line
+	2550 3650 2950 3650
+Connection ~ 2550 3650
+Wire Wire Line
+	1500 3650 2550 3650
+$Comp
+L ArgonComponents:93LCxxA U?
+U 1 1 5FD2093F
+P 2100 4350
+F 0 "U?" H 2100 4700 50  0000 C CNN
+F 1 "93LCxxA" H 2250 4100 50  0000 C CNN
+F 2 "" H 2100 4350 50  0001 C CNN
+F 3 "http://ww1.microchip.com/downloads/en/DeviceDoc/20001749K.pdf" H 2100 4350 50  0001 C CNN
+	1    2100 4350
+	1    0    0    -1
+$EndComp
+Wire Wire Line
+	1500 3650 1500 4150
+Wire Wire Line
+	1400 3650 1500 3650
+Connection ~ 1500 3650
+Wire Wire Line
+	2550 4000 2550 4450
+$Comp
+L Device:R R?
+U 1 1 5FD4899A
+P 3350 3850
+F 0 "R?" H 3250 3850 50  0000 C CNN
+F 1 "10K" V 3450 3850 50  0000 C CNN
+F 2 "" V 3280 3850 50  0001 C CNN
+F 3 "~" H 3350 3850 50  0001 C CNN
+	1    3350 3850
+	-1   0    0    1
+$EndComp
+Wire Wire Line
+	3350 4000 3350 4150
+Wire Wire Line
+	2950 4000 2950 4250
+Wire Wire Line
+	2500 4350 3350 4350
+Wire Wire Line
+	3350 4450 3350 4350
+Connection ~ 3350 4350
+Wire Wire Line
+	3350 4350 4500 4350
+Wire Wire Line
+	3100 4450 3350 4450
+$Comp
+L Device:R R?
+U 1 1 5FD3BE55
+P 2950 4450
+F 0 "R?" V 3000 4250 50  0000 C CNN
+F 1 "2.2K" V 3000 4650 50  0000 C CNN
+F 2 "" V 2880 4450 50  0001 C CNN
+F 3 "~" H 2950 4450 50  0001 C CNN
+	1    2950 4450
+	0    1    1    0
+$EndComp
 $EndSCHEMATC

Commit message: Place 555
Parts:
- added U?: NE555D, Package_SO:SOIC-8_3.9x4.9mm_P1.27mm, symbol Timer:NE555D
Changed lines of the file:
@@
 	0    1    1    0
 $EndComp
+$Comp
+L Timer:NE555D U?
+U 1 1 5FD5C58C
+P 8750 2050
+F 0 "U?" H 8750 2631 50  0000 C CNN
+F 1 "NE555D" H 8750 2540 50  0000 C CNN
+F 2 "Package_SO:SOIC-8_3.9x4.9mm_P1.27mm" H 9600 1650 50  0001 C CNN
+F 3 "http://www.ti.com/lit/ds/symlink/ne555.pdf" H 9600 1650 50  0001 C CNN
+	1    8750 2050
+	1    0    0    -1
+$EndComp
 $EndSCHEMATC

Commit message: Add 555
Parts:
- removed U?: NE555D, Package_SO:SOIC-8_3.9x4.9mm_P1.27mm, symbol Timer:NE555D
- added C?: 1uF, symbol Device:CP1
- added C?: 10uF, symbol Device:C
- added D?: LED, symbol Device:LED
- added R?: 1.5K, symbol Device:R
- added R?: 330, symbol Device:R
- added R?: 100K, symbol Device:R
- added U?: LMC555xM, Package_SO:SOIC-8_3.9x4.9mm_P1.27mm, symbol Timer:LMC555xM
- C? (x2): value C -> 27pF
Connections:
- wire segments 66 -> 93

Commit message: Add LDO
Parts:
- added C? (x2): 1uF, symbol Device:C
- added R?: 12K/1%, symbol Device:R
- added R?: 1K, symbol Device:R
- added U?: MCP1700, Package_TO_SOT_SMD:SOT-23, symbol Regulator_Linear:MCP1700-3302E_SOT23
Connections:
- net VCC is gone; now on net VCC3V3: R?.1, R?.2, R?.2, R?.2, R?.2, U?.4 (R), U?.8 (VCC), U?.8 (VCC)
- net GND: now also C?.1, C?.2, R?.1, U?.1 (GND)
- net at U?.14 (~RESET): now also R?.2
- net VCC3V3: now reaches U?.20 (VCCIO)
- net VCC3V3: now also U?.31 (VCCIO), U?.42 (VCCIO), U?.50 (VREGIN), U?.56 (VCCIO), C?.1, R?.1, U?.2 (VO)
- net at U?.6 (REF): now also R?.2
- net VBUS: now reaches J?.1 (VBUS)
- net VBUS: now also C?.2, U?.3 (VI)
Other:
- moved on the sheet: J?
Changed lines of the file:
@@
 Comment4 ""
 $EndDescr
-Wire Wire Line
-	2300 2650 3750 2650
-NoConn ~ 2300 2750
 $Comp
 L Device:Crystal Y?
@@
 Wire Wire Line
 	5600 5850 5700 5850
-Wire Wire Line
-	3750 2550 2300 2550
 $Comp
 L Device:R R?
@@
 	0    1    1    0
 $EndComp
-Wire Wire Line
-	1900 3050 1950 3050
-Connection ~ 1900 3050
-Wire Wire Line
-	1900 3200 1900 3050
-Wire Wire Line
-	1850 3050 1900 3050
-$Comp
-L power:GND #PWR?
-U 1 1 5FCEE675
-P 1900 3200
-F 0 "#PWR?" H 1900 2950 50  0001 C CNN
-F 1 "GND" H 1905 3027 50  0000 C CNN
-F 2 "" H 1900 3200 50  0001 C CNN
-F 3 "" H 1900 3200 50  0001 C CNN
-	1    1900 3200
-	1    0    0    -1
-$EndComp
-Wire Wire Line
-	1850 3050 1850 2950
-Wire Wire Line
-	1950 2950 1950 3050
 $Comp
 L power:GND #PWR?
@@
 Wire Wire Line
 	1500 4250 1500 4350
-$Comp
-L ArgonComponents:USB_B_Micro J?
-U 1 1 5FCEC245
-P 2000 2550
-F 0 "J?" H 2000 2900 50  0000 C CNN
-F 1 "USB" H 2200 2200 50  0000 R CNN
-F 2 "" H 2150 2400 50  0001 C CNN
-F 3 "~" H 2150 2400 50  0001 C CNN
-	1    2000 2550
-	1    0    0    -1
-$EndComp
 Text GLabel 1400 3650 0    50   Input ~ 0
-VCC
+VCC3V3
 Wire Wire Line
 	1500 4150 1800 4150
@@
 	9250 2050 9250 1800
 Text GLabel 9200 850  0    50   Input ~ 0
-VCC
+VCC3V3
 Wire Wire Line
 	9250 1000 9250 850
@@
 	8750 1600 8600 1600
 Text GLabel 8600 1600 0    50   Input ~ 0
-VCC
+VCC3V3
 Wire Wire Line
 	8750 1200 8550 1200
@@
 $EndComp
 Text GLabel 7700 1000 0    50   Input ~ 0
-VCC
+VCC3V3
 Wire Wire Line
 	7700 1000 8000 1000
@@
 	1    0    0    -1
 $EndComp
-Text GLabel 9600 1950 0    50   Input ~ 0
-VCC
+Text GLabel 9650 1950 0    50   Input ~ 0
+VCC3V3
 $Comp
 L Device:R R?
@@
 $EndComp
 Wire Wire Line
-	9800 1950 9600 1950
+	9800 1950 9650 1950
 Wire Wire Line
 	11000 1950 11000 2100
@@
 $EndComp
 Wire Wire Line
-	4050 2650 4500 2650
-Wire Wire Line
-	4500 2550 4050 2550
-Wire Wire Line
 	3350 4150 4500 4150
 Wire Wire Line
@@
 Wire Wire Line
 	5300 5650 5300 5850
-$Comp
-L Interface_USB:FT2232HL U?
-U 1 1 5FC7546A
-P 5700 3450
-F 0 "U?" H 5700 5831 50  0000 C CNN
-F 1 "FT2232HL" H 5700 5740 50  0000 C CNN
-F 2 "Package_QFP:LQFP-64_10x10mm_P0.5mm" H 5700 3450 50  0001 C CNN
-F 3 "https://www.ftdichip.com/Support/Documents/DataSheets/ICs/DS_FT2232H.pdf" H 5700 3450 50  0001 C CNN
-	1    5700 3450
-	1    0    0    -1
-$EndComp
 Wire Wire Line
 	4400 5850 5100 5850
@@
 	0    1    1    0
 $EndComp
+Text GLabel 3700 1750 0    50   Input ~ 0
+VCORE
+Wire Wire Line
+	6200 800  6200 1250
+Connection ~ 6100 800
+Wire Wire Line
+	6100 800  6200 800
+Wire Wire Line
+	6100 800  6100 1250
+Wire Wire Line
+	6000 1250 6000 800
+Wire Wire Line
+	6400 800  6200 800
+Connection ~ 6000 800
+Wire Wire Line
+	6000 800  6100 800
+Wire Wire Line
+	5900 800  6000 800
+Wire Wire Line
+	5900 800  5900 1250
+Connection ~ 6200 800
+Text GLabel 6400 800  2    50   Input ~ 0
+VCC3V3
+$Comp
+L Regulator_Linear:MCP1700-3302E_SOT23 U?
+U 1 1 5FD82696
+P 1750 1100
+F 0 "U?" H 1900 850 50  0000 C CNN
+F 1 "MCP1700" H 1750 1250 50  0000 C CNN
+F 2 "Package_TO_SOT_SMD:SOT-23" H 1750 1325 50  0001 C CNN
+F 3 "http://ww1.microchip.com/downloads/en/DeviceDoc/20001826D.pdf" H 1750 1100 50  0001 C CNN
+	1    1750 1100
+	1    0    0    -1
+$EndComp
+Wire Wire Line
+	4050 2650 4500 2650
+Wire Wire Line
+	4500 2550 4050 2550
+Wire Wire Line
+	3100 2350 2950 2350
+Text GLabel 3100 2350 2    50   Input ~ 0
+VBUS
+NoConn ~ 2950 2750
+Wire Wire Line
+	2550 3050 2600 3050
+Connection ~ 2550 3050
+Wire Wire Line
+	2550 3200 2550 3050
+Wire Wire Line
+	2500 3050 2550 3050
+$Comp
+L power:GND #PWR?
+U 1 1 5FCEE675
+P 2550 3200
+F 0 "#PWR?" H 2550 2950 50  0001 C CNN
+F 1 "GND" H 2555 3027 50  0000 C CNN
+F 2 "" H 2550 3200 50  0001 C CNN
+F 3 "" H 2550 3200 50  0001 C CNN
+	1    2550 3200
+	1    0    0    -1
+$EndComp
+Wire Wire Line
+	2500 3050 2500 2950
+Wire Wire Line
+	2600 2950 2600 3050
+$Comp
+L ArgonComponents:USB_B_Micro J?
+U 1 1 5FCEC245
+P 2650 2550
+F 0 "J?" H 2650 2900 50  0000 C CNN
+F 1 "USB" H 2850 2200 50  0000 R CNN
+F 2 "" H 2800 2400 50  0001 C CNN
+F 3 "~" H 2800 2400 50  0001 C CNN
+	1    2650 2550
+	1    0    0    -1
+$EndComp
+Wire Wire Line
+	2950 2650 3750 2650
+Text GLabel 950  1100 0    50   Input ~ 0
+VBUS
+Wire Wire Line
+	950  1100 1150 1100
+Wire Wire Line
+	1750 1400 1750 1500
+Wire Wire Line
+	1150 1100 1150 1500
+Connection ~ 1150 1100
+Wire Wire Line
+	1150 1100 1450 1100
+Wire Wire Line
+	2350 1100 2350 1500
+Wire Wire Line
+	2050 1100 2350 1100
+Connection ~ 2350 1100
+Wire Wire Line
+	2350 1100 2550 1100
+$Comp
+L Device:C C?
+U 1 1 5FDB6529
+P 1350 1500
+F 0 "C?" V 1300 1600 50  0000 C CNN
+F 1 "1uF" V 1400 1650 50  0000 C CNN
+F 2 "" H 1388 1350 50  0001 C CNN
+F 3 "~" H 1350 1500 50  0001 C CNN
+	1    1350 1500
+	0    1    1    0
+$EndComp
+Wire Wire Line
+	1500 1500 1750 1500
+Connection ~ 1750 1500
+Wire Wire Line
+	1750 1500 1750 1800
+$Comp
+L power:GND #PWR?
+U 1 1 5FD8357B
+P 1750 1800
+F 0 "#PWR?" H 1750 1550 50  0001 C CNN
+F 1 "GND" H 1755 1627 50  0000 C CNN
+F 2 "" H 1750 1800 50  0001 C CNN
+F 3 "" H 1750 1800 50  0001 C CNN
+	1    1750 1800
+	1    0    0    -1
+$EndComp
+Wire Wire Line
+	1950 1500 1750 1500
+Wire Wire Line
+	2350 1500 2250 1500
+$Comp
+L Device:C C?
+U 1 1 5FDB5C8F
+P 2100 1500
+F 0 "C?" V 2050 1600 50  0000 C CNN
+F 1 "1uF" V 2150 1650 50  0000 C CNN
+F 2 "" H 2138 1350 50  0001 C CNN
+F 3 "~" H 2100 1500 50  0001 C CNN
+	1    2100 1500
+	0    1    1    0
+$EndComp
+Wire Wire Line
+	1200 1500 1150 1500
+Text GLabel 2550 1100 2    50   Input ~ 0
+VCC3V3
+Wire Wire Line
+	2950 2550 3750 2550
+Wire Wire Line
+	4500 2850 3750 2850
+Wire Wire Line
+	4500 1550 4200 1550
+Text GLabel 4200 1550 0    50   Input ~ 0
+VCC3V3
+Wire Wire Line
+	3750 2850 3750 2950
+Wire Wire Line
+	3750 3250 3750 3350
+$Comp
+L Device:R R?
+U 1 1 5FDEBE59
+P 3750 3100
+F 0 "R?" H 3650 3100 50  0000 C CNN
+F 1 "12K/1%" V 3850 3100 50  0000 C CNN
+F 2 "" V 3680 3100 50  0001 C CNN
+F 3 "~" H 3750 3100 50  0001 C CNN
+	1    3750 3100
+	-1   0    0    1
+$EndComp
+$Comp
+L power:GND #PWR?
+U 1 1 5FDEBBC5
+P 3750 3350
+F 0 "#PWR?" H 3750 3100 50  0001 C CNN
+F 1 "GND" H 3755 3177 50  0000 C CNN
+F 2 "" H 3750 3350 50  0001 C CNN
+F 3 "" H 3750 3350 50  0001 C CNN
+	1    3750 3350
+	1    0    0    -1
+$EndComp
+Wire Wire Line
+	4150 3450 4150 3550
+$Comp
+L Device:R R?
+U 1 1 5FE11A95
+P 4150 3300
+F 0 "R?" H 4050 3300 50  0000 C CNN
+F 1 "1K" V 4250 3300 50  0000 C CNN
+F 2 "" V 4080 3300 50  0001 C CNN
+F 3 "~" H 4150 3300 50  0001 C CNN
+	1    4150 3300
+	-1   0    0    1
+$EndComp
+Wire Wire Line
+	4150 3050 4150 3150
+$Comp
+L Interface_USB:FT2232HL U?
+U 1 1 5FC7546A
+P 5700 3450
+F 0 "U?" H 6700 5550 50  0000 C CNN
+F 1 "FT2232HL" H 6550 1350 50  0000 C CNN
+F 2 "Package_QFP:LQFP-64_10x10mm_P0.5mm" H 5700 3450 50  0001 C CNN
+F 3 "https://www.ftdichip.com/Support/Documents/DataSheets/ICs/DS_FT2232H.pdf" H 5700 3450 50  0001 C CNN
+	1    5700 3450
+	1    0    0    -1
+$EndComp
+Wire Wire Line
+	4500 3050 4150 3050
+Text GLabel 4150 3550 3    50   Input ~ 0
+VCC3V3
 $EndSCHEMATC

Commit message: Chaotic evil - argon, benzen, some random freecad
Parts:
- added J2: V3V3-GND, Connector_PinHeader_2.54mm:PinHeader_1x02_P2.54mm_Vertical, symbol ArgonComponents:V3V3-GND
- added S1, S3: Connector8, Connector_PinHeader_2.54mm:PinHeader_1x08_P2.54mm_Vertical, symbol ArgonComponents:Connector8
- added S2, S4: Connector8_FTDI, Connector_PinHeader_2.54mm:PinHeader_1x08_P2.54mm_Vertical, symbol ArgonComponents:Connector8_FTDI
- C1, C2, C3, C4, C5, C6: renamed from C?; footprint (none) -> Capacitor_SMD:C_0603_1608Metric
- D1: renamed from D?; footprint (none) -> LED_SMD:LED_0603_1608Metric
- J1: renamed from J?; footprint (none) -> Connector_USB:USB_Mini-B_AdamTech_MUSB-B5-S-VT-TSMT-1_SMD_Vertical
- R1, R10, R11, R2, R3, R4, R5, R6, R7, R8, R9: renamed from R?; footprint (none) -> Resistor_SMD:R_0603_1608Metric
- U2: renamed from U?; footprint (none) -> Package_SO:SOIC-8_3.9x4.9mm_P1.27mm
- Y1: renamed from Y?; footprint (none) -> Crystal:Crystal_SMD_SeikoEpson_TSX3225-4Pin_3.2x2.5mm
- gave numbers to parts that had none: 3
Connections:
- net GND: now also J2.1 (GND)
- net VCC3V3: now also J2.2 (V3V3)
- net at U3.16 (ADBUS0): now also S1.1 (0), S2.1 (0)
- net at U3.17 (ADBUS1): now also S1.2 (1), S2.2 (1)
- net at U3.18 (ADBUS2): now also S1.3 (2), S2.3 (2)
- net at U3.19 (ADBUS3): now also S1.4 (3), S2.4 (3)
- net at U3.21 (ADBUS4): now also S1.5 (4), S2.5 (4)
- net at U3.22 (ADBUS5): now also S1.6 (5), S2.6 (5)
- net at U3.23 (ADBUS6): now also S1.7 (6), S2.7 (6)
- net at U3.24 (ADBUS7): now also S1.8 (7), S2.8 (7)
- net at U3.38 (BDBUS0): now also S3.1 (0), S4.1 (0)
- net at U3.39 (BDBUS1): now also S3.2 (1), S4.2 (1)
- net at U3.40 (BDBUS2): now also S3.3 (2), S4.3 (2)
- net at U3.41 (BDBUS3): now also S3.4 (3), S4.4 (3)
- net at U3.43 (BDBUS4): now also S3.5 (4), S4.5 (4)
- net at U3.44 (BDBUS5): now also S3.6 (5), S4.6 (5)
- net at U3.45 (BDBUS6): now also S3.7 (6), S4.7 (6)
- net at U3.46 (BDBUS7): now also S3.8 (7), S4.8 (7)
- no-connect marks 1 -> 13
Other:
- note added: "LED RX"
- note added: "LED TX"
- moved on the sheet: C5, C6, D1, R10, R11, R9, U4

Commit message: Argon USB & custom footprint for DIP-16
Parts:
- J1: footprint Connector_USB:USB_Mini-B_AdamTech_MUSB-B5-S-VT-TSMT-1_SMD_Vertical -> Connector_USB:USB_Mini-B_Wuerth_65100516121_Horizontal
Changed lines of the file:
@@
 F 0 "J1" H 2650 2900 50  0000 C CNN
 F 1 "USB" H 2850 2200 50  0000 R CNN
-F 2 "Connector_USB:USB_Mini-B_AdamTech_MUSB-B5-S-VT-TSMT-1_SMD_Vertical" H 2800 2400 50  0001 C CNN
+F 2 "Connector_USB:USB_Mini-B_Wuerth_65100516121_Horizontal" H 2800 2400 50  0001 C CNN
 F 3 "~" H 2800 2400 50  0001 C CNN
 	1    2650 2550

Commit message: Aegon USB and power
Parts:
- removed C1: 1uF, Capacitor_SMD:C_0603_1608Metric, symbol Device:C
- removed U1: MCP1700, Package_TO_SOT_SMD:SOT-23, symbol Regulator_Linear:MCP1700-3302E_SOT23
- added C?: 10nF, Capacitor_SMD:C_0603_1608Metric, symbol Device:C
- added C?: 100nF, Capacitor_SMD:C_0603_1608Metric, symbol Device:C
- added C?: 22uF, Capacitor_SMD:C_0603_1608Metric, symbol Device:C
- added D?: LED, symbol Device:LED
- added R?: 120R, Resistor_SMD:R_0603_1608Metric, symbol Device:R
- added R?: 100R, Resistor_SMD:R_0603_1608Metric, symbol Device:R
- added U?: AMS1117-3.3, Package_TO_SOT_SMD:SOT-223-3_TabPin2, symbol Regulator_Linear:AMS1117-3.3
- C2: value 1uF -> 100uF
Connections:
- net labels added: V3V3
- net labels removed: VBUS
- wire segments 174 -> 177
Other:
- note added: "LDO voltage regulator"
- moved on the sheet: C2, C3, C4, C5, C6, D1, J1, J2, R1, R10, R11, R2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

Commit message: More voltages
Parts:
- added C? (x3): 4.7uF, Capacitor_SMD:C_0603_1608Metric, symbol Device:CP1
- added C? (x10): 100nF, Capacitor_SMD:C_0603_1608Metric, symbol Device:C
- added D?: LED, symbol Device:LED
- added FB? (x2): 600R/0.5A, symbol Device:Ferrite_Bead_Small
- added R?: 220R, Resistor_SMD:R_0603_1608Metric, symbol Device:R
- R?: value 100R -> 220R
Connections:
- net labels added: LED_RX_A, LED_RX_B, LED_TX_A, LED_TX_B
- wire segments 177 -> 260
Other:
- note added: "EEPROM"
- note removed: "LED RX"
- note removed: "LED TX"
- moved on the sheet: C2, C3, C4, C5, C6, C?, D1, D?, J1, J2, R1, R10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
