File: argon/argon.sch (KiCad schematic (older format))
At the start: 51 parts, among them J1 USB, J2 V3V3-GND, U2 93LCxxA, U3 FT2232HL, U4 LMC555xM, Y1 12Mhz

Commit message: Leds & structure
Parts:
- added D? (x3): LED, symbol Device:LED
- added R? (x3): 220R, Resistor_SMD:R_0603_1608Metric, symbol Device:R
Connections:
- wire segments 260 -> 265
- no-connect marks 13 -> 15
Other:
- moved on the sheet: C2, C3, C4, C5, C6, C?, D1, D?, FB?, J1, J2, R1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

Commit message: Fix bugs
Parts:
- removed FB? (x2): 600R/0.5A, symbol Device:Ferrite_Bead_Small
- added C17: 1uF, Capacitor_SMD:C_0603_1608Metric, symbol Device:CP1
- added C9: 10uF, Capacitor_SMD:C_0603_1608Metric, symbol Device:C
- added D3: LED, LED_SMD:LED_0603_1608Metric, symbol Device:LED
- added FB1, FB2: 600R/0.5A, symbol ArgonComponents:Ferrite_Bead
- added J3: V3V3-GND, Connector_PinHeader_2.54mm:PinHeader_1x02_P2.54mm_Vertical, symbol ArgonComponents:V3V3-GND
- added R10: 1.5K, Resistor_SMD:R_0603_1608Metric, symbol Device:R
- added R15: 100K, Resistor_SMD:R_0603_1608Metric, symbol Device:R
- added R16: 330R, Resistor_SMD:R_0603_1608Metric, symbol Device:R
- added U4: LMC555xM, Package_SO:SOIC-8_3.9x4.9mm_P1.27mm, symbol Timer:LMC555xM
- R4: renamed from R11; value 330 -> 330R
- gave numbers to parts that had none: 28
- renumbered C3 to C10, C4 to C11, C5 to C3, C2 to C4, R9 to R1, R5 to R11, R6 to R12, R7 to R13, R8 to R14, R10 to R3, R1 to R5, R2 to R7, R3 to R8, R4 to R9, S3 to S2, S2 to S3, U4 to U1, U2 to U3, U3 to U5
Connections:
- net VCC3V3 is gone; now on net V3V3: J2.2 (V3V3), R5.2, R7.2, R9.2
- net GND: now also U3.5 (GND), U5.1 (GND), U5.10 (AGND), U5.11 (GND), U5.15 (GND), U5.25 (GND), U5.35 (GND), U5.47 (GND), U5.5 (GND), U5.51 (GND), C17.2, C9.2, D3.1 (K), J3.1 (GND), U4.1 (GND); no longer C1.2, C2.2, R2.1
- net V3V3: now also U3.8 (VCC), FB1.2, FB2.2, J3.2 (V3V3), R10.2, R15.1, U4.4 (R), U4.8 (VCC)
- net CS_A: now reaches S1.4 (3), S3.4 (3), U5.19 (ADBUS3)
- net CS_A: now also R1.1, U1.2 (TR)
- net at C13.1, C15.2, U5.4 (VPHY): now also FB2.1
- net CS_B: now reaches S2.4 (3), S4.4 (3), U5.41 (BDBUS3)
- net CS_B: now also R10.1, U4.2 (TR)
- net at C12.1, C14.2, U5.9 (VPLL): now also FB1.1
- net at J1.6 (Shield): now also C1.2, C2.2, R2.1
- new net: D3.2 (A), R16.1
- new net: R16.2, U4.3 (Q)
- new net: C17.1, R15.2, U4.6 (THR), U4.7 (DIS)
- new net: C9.1, U4.5 (CV)
Other:
- moved on the sheet: C1, C10, C11, C12, C13, C14, C15, C16, C18, C19, C2, C20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

Commit message: Final schematic
Parts:
- added C24: 100nF, Capacitor_SMD:C_0603_1608Metric, symbol Device:C
- C4: value 100uF -> 100nF
- R11: value 12K/1% -> 12K
Connections:
- net GND: now also C24.1
- net V3V3: now also C24.2
Other:
- moved on the sheet: C12, C14, FB1, FB2, R5, R7, R8, R9, U3

Commit message: Add FBs and start positioning buses on PCB
Parts:
- added J4, J5: V3V3-GND, Connector_PinHeader_2.54mm:PinHeader_1x02_P2.54mm_Vertical, symbol ArgonComponents:V3V3-GND
- D1, D3: footprint LED_SMD:LED_0603_1608Metric -> LED_SMD:LED_0805_2012Metric
- D2, D4, D5, D6, D7: footprint (none) -> LED_SMD:LED_0805_2012Metric
- FB1, FB2: footprint (none) -> FBead_Murata_BLM18AG601SN1D:Murata-BLM18-0.15-t0.8-0-0-IPC_A
Connections:
- net GND: now also J4.1 (GND), J5.1 (GND)
- net V3V3: now also J4.2 (V3V3), J5.2 (V3V3)
Changed lines of the file:
@@
 F 0 "D1" H 4650 9550 50  0000 C CNN
 F 1 "LED" H 4650 9750 50  0000 C CNN
-F 2 "LED_SMD:LED_0603_1608Metric" H 4650 9650 50  0001 C CNN
+F 2 "LED_SMD:LED_0805_2012Metric" H 4650 9650 50  0001 C CNN
 F 3 "~" H 4650 9650 50  0001 C CNN
 	1    4650 9650
@@
 F 0 "D4" H 14350 1150 50  0000 C CNN
 F 1 "LED" H 14350 1400 50  0000 C CNN
-F 2 "" H 14350 1250 50  0001 C CNN
+F 2 "LED_SMD:LED_0805_2012Metric" H 14350 1250 50  0001 C CNN
 F 3 "~" H 14350 1250 50  0001 C CNN
 	1    14350 1250
@@
 F 0 "D5" H 14350 1550 50  0000 C CNN
 F 1 "LED" H 14350 1800 50  0000 C CNN
-F 2 "" H 14350 1650 50  0001 C CNN
+F 2 "LED_SMD:LED_0805_2012Metric" H 14350 1650 50  0001 C CNN
 F 3 "~" H 14350 1650 50  0001 C CNN
 	1    14350 1650
@@
 F 0 "D6" H 14350 1950 50  0000 C CNN
 F 1 "LED" H 14350 2200 50  0000 C CNN
-F 2 "" H 14350 2050 50  0001 C CNN
+F 2 "LED_SMD:LED_0805_2012Metric" H 14350 2050 50  0001 C CNN
 F 3 "~" H 14350 2050 50  0001 C CNN
 	1    14350 2050
@@
 F 0 "D7" H 14350 2350 50  0000 C CNN
 F 1 "LED" H 14350 2600 50  0000 C CNN
-F 2 "" H 14350 2450 50  0001 C CNN
+F 2 "LED_SMD:LED_0805_2012Metric" H 14350 2450 50  0001 C CNN
 F 3 "~" H 14350 2450 50  0001 C CNN
 	1    14350 2450
@@
 F 0 "D3" H 8850 9550 50  0000 C CNN
 F 1 "LED" H 8850 9750 50  0000 C CNN
-F 2 "LED_SMD:LED_0603_1608Metric" H 8850 9650 50  0001 C CNN
+F 2 "LED_SMD:LED_0805_2012Metric" H 8850 9650 50  0001 C CNN
 F 3 "~" H 8850 9650 50  0001 C CNN
 	1    8850 9650
@@
 F 0 "D2" H 5950 3050 50  0000 C CNN
 F 1 "LED" H 5950 3300 50  0000 C CNN
-F 2 "" H 5950 3150 50  0001 C CNN
+F 2 "LED_SMD:LED_0805_2012Metric" H 5950 3150 50  0001 C CNN
 F 3 "~" H 5950 3150 50  0001 C CNN
 	1    5950 3150
@@
 F 0 "FB2" V 5850 2300 50  0000 C CNN
 F 1 "600R/0.5A" V 6150 2300 50  0000 C CNN
-F 2 "" V 5930 2300 50  0001 C CNN
+F 2 "FBead_Murata_BLM18AG601SN1D:Murata-BLM18-0.15-t0.8-0-0-IPC_A" V 5930 2300 50  0001 C CNN
 F 3 "~" H 6000 2300 50  0001 C CNN
 	1    6000 2300
@@
 F 0 "FB1" V 5850 1300 50  0000 C CNN
 F 1 "600R/0.5A" V 6150 1300 50  0000 C CNN
-F 2 "" V 5930 1300 50  0001 C CNN
+F 2 "FBead_Murata_BLM18AG601SN1D:Murata-BLM18-0.15-t0.8-0-0-IPC_A" V 5930 1300 50  0001 C CNN
 F 3 "~" H 6000 1300 50  0001 C CNN
 	1    6000 1300
@@
 Wire Wire Line
 	8050 2300 8050 3700
+$Comp
+L ArgonComponents:V3V3-GND J4
+U 1 1 61468AEA
+P 13050 8000
+F 0 "J4" H 12967 7777 50  0000 C CNN
+F 1 "V3V3-GND" H 13050 7800 50  0001 C CNN
+F 2 "Connector_PinHeader_2.54mm:PinHeader_1x02_P2.54mm_Vertical" H 13050 8000 50  0001 C CNN
+F 3 "~" H 13050 8000 50  0001 C CNN
+	1    13050 8000
+	-1   0    0    1
+$EndComp
+Wire Wire Line
+	13350 8000 13550 8000
+Wire Wire Line
+	13550 8000 13550 8100
+Wire Wire Line
+	13350 7900 13550 7900
+$Comp
+L power:GND #PWR0102
+U 1 1 61468AF3
+P 13550 8100
+F 0 "#PWR0102" H 13550 7850 50  0001 C CNN
+F 1 "GND" H 13555 7927 50  0000 C CNN
+F 2 "" H 13550 8100 50  0001 C CNN
+F 3 "" H 13550 8100 50  0001 C CNN
+	1    13550 8100
+	1    0    0    -1
+$EndComp
+Text GLabel 13550 7900 2    50   Input ~ 0
+V3V3
+$Comp
+L ArgonComponents:V3V3-GND J5
+U 1 1 61468AFA
+P 13050 8800
+F 0 "J5" H 12967 8577 50  0000 C CNN
+F 1 "V3V3-GND" H 13050 8600 50  0001 C CNN
+F 2 "Connector_PinHeader_2.54mm:PinHeader_1x02_P2.54mm_Vertical" H 13050 8800 50  0001 C CNN
+F 3 "~" H 13050 8800 50  0001 C CNN
+	1    13050 8800
+	-1   0    0    1
+$EndComp
+Wire Wire Line
+	13350 8800 13550 8800
+Wire Wire Line
+	13550 8800 13550 8900
+Wire Wire Line
+	13350 8700 13550 8700
+$Comp
+L power:GND #PWR0103
+U 1 1 61468B03
+P 13550 8900
+F 0 "#PWR0103" H 13550 8650 50  0001 C CNN
+F 1 "GND" H 13555 8727 50  0000 C CNN
+F 2 "" H 13550 8900 50  0001 C CNN
+F 3 "" H 13550 8900 50  0001 C CNN
+	1    13550 8900
+	1    0    0    -1
+$EndComp
+Text GLabel 13550 8700 2    50   Input ~ 0
+V3V3
 $EndSCHEMATC
