File: argon/_autosave-argon.sch (KiCad schematic (older format))
At the start: 72 parts, among them J1 USB, J2 V3V3-GND, J3 V3V3-GND, J4 V3V3-GND, J5 V3V3-GND, U1 LMC555xM, U2 AMS1117-3.3, U3 93LCxxA, U4 LMC555xM, U5 FT2232HL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

Commit message: Clear folders
Parts:
- gave numbers to parts that had none: 4
Changed lines of the file:
@@
 Connection ~ 8500 10050
 $Comp
-L Mechanical:MountingHole H?
+L Mechanical:MountingHole H1
 U 1 1 5FE6D4CE
 P 15050 8050
-F 0 "H?" H 15150 8096 50  0000 L CNN
+F 0 "H1" H 15150 8096 50  0000 L CNN
 F 1 "MountingHole" H 15150 8005 50  0000 L CNN
 F 2 "" H 15050 8050 50  0001 C CNN
@@
 $EndComp
 $Comp
-L Mechanical:MountingHole H?
+L Mechanical:MountingHole H2
 U 1 1 5FE6DED5
 P 15050 8300
-F 0 "H?" H 15150 8346 50  0000 L CNN
+F 0 "H2" H 15150 8346 50  0000 L CNN
 F 1 "MountingHole" H 15150 8255 50  0000 L CNN
 F 2 "" H 15050 8300 50  0001 C CNN
@@
 $EndComp
 $Comp
-L Mechanical:MountingHole H?
+L Mechanical:MountingHole H3
 U 1 1 5FE6E061
 P 15050 8550
-F 0 "H?" H 15150 8596 50  0000 L CNN
+F 0 "H3" H 15150 8596 50  0000 L CNN
 F 1 "MountingHole" H 15150 8505 50  0000 L CNN
 F 2 "" H 15050 8550 50  0001 C CNN
@@
 $EndComp
 $Comp
-L Mechanical:MountingHole H?
+L Mechanical:MountingHole H4
 U 1 1 5FE6E20D
 P 15050 8800
-F 0 "H?" H 15150 8846 50  0000 L CNN
+F 0 "H4" H 15150 8846 50  0000 L CNN
 F 1 "MountingHole" H 15150 8755 50  0000 L CNN
 F 2 "" H 15050 8800 50  0001 C CNN
