File: argon/argon.kicad_pcb (KiCad board)
At the start: 2 copper layers, 60 x 50 mm, 78 parts, among them J1 USB, J2 V3V3-GND, J3 V3V3-GND, J4 V3V3-GND, J5 V3V3-GND, J6 V3V3-GND, J7 V3V3-GND, U1 LMC555xM, U2 AMS1117-3.3, U3 93LCxxA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

Commit message: PCB wip
Parts:
- moved C18 55.9 mm to (150.0, 122.2)
- moved C24 14.9 mm to (158.8, 91.4)
- moved C15 5.78 mm to (129.3, 103.9)
- moved C8 3.11 mm to (150.0, 124.2)
- moved FB1 2.76 mm to (129.3, 97.9)
- moved U3 2.70 mm to (165.1, 90.8)
- moved R5 2.70 mm to (171.5, 93.3)
- moved R7 2.70 mm to (171.5, 89.5)
- moved R8 2.70 mm to (171.5, 91.4)
- moved R9 2.70 mm to (171.5, 87.6)
- moved C14 1.08 mm to (170.7, 103.9)
- moved C16 1.00 mm to (150.0, 120.1)
- moved C20 1.00 mm to (150.0, 118.1)
- moved C7 1.00 mm to (150.0, 115.2)
- moved FB2 0.90 mm to (170.7, 97.9)
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Routing:
- net Net-(J1-Pad3): track 9.56 -> 0.00 mm
- net Net-(J1-Pad2): track 5.24 -> 0.00 mm
Changed lines of the file:
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@@
     (thickness 1.6)
     (drawings 49)
-    (tracks 124)
+    (tracks 114)
     (zones 0)
     (modules 78)
@@
   )
   (module Capacitor_Tantalum_SMD:CP_EIA-3216-18_Kemet-A (layer B.Cu)
-    (at 129.968 101.53 180)
+    (at 130 100.92 180)
     (descr "Tantalum Capacitor SMD Kemet-A (3216-18 Metric), IPC_7351 nominal, (Body size from: http://www.kemet.com/Lists/ProductCatalog/Attachments/253/KEM_TC101_STD.pdf), generated with kicad-footprint-generator")
     (tags "capacitor tantalum")
@@
   )
   (module Capacitor_Tantalum_SMD:CP_EIA-3216-18_Kemet-A (layer B.Cu)
-    (at 169.968 101.53)
+    (at 170 100.92)
     (descr "Tantalum Capacitor SMD Kemet-A (3216-18 Metric), IPC_7351 nominal, (Body size from: http://www.kemet.com/Lists/ProductCatalog/Attachments/253/KEM_TC101_STD.pdf), generated with kicad-footprint-generator")
     (tags "capacitor tantalum")
@@
   )
   (module Capacitor_Tantalum_SMD:CP_EIA-3216-18_Kemet-A (layer B.Cu)
-    (at 149.987 114.173 180)
+    (at 149.987 115.173 180)
     (descr "Tantalum Capacitor SMD Kemet-A (3216-18 Metric), IPC_7351 nominal, (Body size from: http://www.kemet.com/Lists/ProductCatalog/Attachments/253/KEM_TC101_STD.pdf), generated with kicad-footprint-generator")
     (tags "capacitor tantalum")
@@
   )
   (module FBead_Murata_BLM18AG601SN1D:Murata-BLM18-0.15-t0.8-0-0-IPC_A (layer B.Cu)
-    (at 170 98.5)
+    (at 170.688 97.92)
     (fp_text reference FB2 (at 1.958 -0.018) (layer B.SilkS)
       (effects (font (size 0.7 0.7) (thickness 0.15)) (justify right mirror))
@@
   )
   (module FBead_Murata_BLM18AG601SN1D:Murata-BLM18-0.15-t0.8-0-0-IPC_A (layer B.Cu)
-    (at 130 95.25 180)
+    (at 129.286 97.92 180)
     (fp_text reference FB1 (at 1.73 0) (layer B.SilkS)
       (effects (font (size 0.7 0.7) (thickness 0.15)) (justify left mirror))
@@
   )
   (module Capacitor_SMD:C_0603_1608Metric (layer B.Cu)
-    (at 173.482 93.472)
+    (at 158.75 91.44)
     (descr "Capacitor SMD 0603 (1608 Metric), square (rectangular) end terminal, IPC_7351 nominal, (Body size source: http://www.tortai-tech.com/upload/download/2011102023233369053.pdf), generated with kicad-footprint-generator")
     (tags capacitor)
     (attr smd)
-    (fp_text reference C24 (at 2.794 0) (layer B.SilkS)
+    (fp_text reference C24 (at 0 -1.27) (layer B.SilkS)
       (effects (font (size 0.7 0.7) (thickness 0.15)) (justify mirror))
     )
@@
     (tags capacitor)
     (attr smd)
-    (fp_text reference C21 (at -2.54 0) (layer B.SilkS)
+    (fp_text reference C21 (at 0 -1.08) (layer B.SilkS)
       (effects (font (size 0.7 0.7) (thickness 0.15)) (justify mirror))
     )
@@
   )
   (module Capacitor_SMD:C_0603_1608Metric (layer B.Cu)
-    (at 149.987 117.094)
+    (at 149.987 118.094)
     (descr "Capacitor SMD 0603 (1608 Metric), square (rectangular) end terminal, IPC_7351 nominal, (Body size source: http://www.tortai-tech.com/upload/download/2011102023233369053.pdf), generated with kicad-footprint-generator")
     (tags capacitor)
@@
     (tags capacitor)
     (attr smd)
-    (fp_text reference C19 (at 2.54 0) (layer B.SilkS)
+    (fp_text reference C19 (at 0 -1.08) (layer B.SilkS)
       (effects (font (size 0.7 0.7) (thickness 0.15)) (justify mirror))
     )
@@
   )
   (module Capacitor_SMD:C_0603_1608Metric (layer B.Cu)
-    (at 205.359 114.3)
+    (at 149.987 122.174)
     (descr "Capacitor SMD 0603 (1608 Metric), square (rectangular) end terminal, IPC_7351 nominal, (Body size source: http://www.tortai-tech.com/upload/download/2011102023233369053.pdf), generated with kicad-footprint-generator")
     (tags capacitor)
     (attr smd)
-    (fp_text reference C18 (at 0 1.43) (layer B.SilkS)
+    (fp_text reference C18 (at -2.413 0) (layer B.SilkS)
       (effects (font (size 0.7 0.7) (thickness 0.15)) (justify mirror))
     )
@@
   )
   (module Capacitor_SMD:C_0603_1608Metric (layer B.Cu)
-    (at 149.987 119.094)
+    (at 149.987 120.094)
     (descr "Capacitor SMD 0603 (1608 Metric), square (rectangular) end terminal, IPC_7351 nominal, (Body size source: http://www.tortai-tech.com/upload/download/2011102023233369053.pdf), generated with kicad-footprint-generator")
     (tags capacitor)
@@
   )
   (module Capacitor_SMD:C_0603_1608Metric (layer B.Cu)
-    (at 130 98.188)
+    (at 129.286 103.92)
     (descr "Capacitor SMD 0603 (1608 Metric), square (rectangular) end terminal, IPC_7351 nominal, (Body size source: http://www.tortai-tech.com/upload/download/2011102023233369053.pdf), generated with kicad-footprint-generator")
     (tags capacitor)
@@
   )
   (module Capacitor_SMD:C_0603_1608Metric (layer B.Cu)
-    (at 169.926 104.648 180)
+    (at 170.688 103.886 180)
     (descr "Capacitor SMD 0603 (1608 Metric), square (rectangular) end terminal, IPC_7351 nominal, (Body size source: http://www.tortai-tech.com/upload/download/2011102023233369053.pdf), generated with kicad-footprint-generator")
     (tags capacitor)
@@
   )
   (module Capacitor_SMD:C_0603_1608Metric (layer B.Cu)
-    (at 149.987 121.094)
+    (at 149.987 124.206)
     (descr "Capacitor SMD 0603 (1608 Metric), square (rectangular) end terminal, IPC_7351 nominal, (Body size source: http://www.tortai-tech.com/upload/download/2011102023233369053.pdf), generated with kicad-footprint-generator")
     (tags capacitor)
@@
     (tags capacitor)
     (attr smd)
-    (fp_text reference C5 (at 0 1.43) (layer B.SilkS)
+    (fp_text reference C5 (at 0 -1.16) (layer B.SilkS)
       (effects (font (size 0.7 0.7) (thickness 0.15)) (justify mirror))
     )
@@
   )
   (module Package_SO:SOIC-8_3.9x4.9mm_P1.27mm (layer B.Cu)
-    (at 167.132 89.004 180)
+    (at 165.1 90.782 180)
     (descr "SOIC, 8 Pin (JEDEC MS-012AA, https://www.analog.com/media/en/package-pcb-resources/package/pkg_pdf/soic_narrow-r/r_8.pdf), generated with kicad-footprint-generator ipc_gullwing_generator.py")
     (tags "SOIC SO")
@@
   )
   (module Resistor_SMD:R_0603_1608Metric (layer B.Cu)
-    (at 173.5075 85.805)
+    (at 171.4755 87.583)
     (descr "Resistor SMD 0603 (1608 Metric), square (rectangular) end terminal, IPC_7351 nominal, (Body size source: http://www.tortai-tech.com/upload/download/2011102023233369053.pdf), generated with kicad-footprint-generator")
     (tags resistor)
@@
   )
   (module Resistor_SMD:R_0603_1608Metric (layer B.Cu)
-    (at 173.5075 89.615 180)
+    (at 171.4755 91.393 180)
     (descr "Resistor SMD 0603 (1608 Metric), square (rectangular) end terminal, IPC_7351 nominal, (Body size source: http://www.tortai-tech.com/upload/download/2011102023233369053.pdf), generated with kicad-footprint-generator")
     (tags resistor)
@@
   )
   (module Resistor_SMD:R_0603_1608Metric (layer B.Cu)
-    (at 173.5075 87.71)
+    (at 171.4755 89.488)
     (descr "Resistor SMD 0603 (1608 Metric), square (rectangular) end terminal, IPC_7351 nominal, (Body size source: http://www.tortai-tech.com/upload/download/2011102023233369053.pdf), generated with kicad-footprint-generator")
     (tags resistor)
@@
   )
   (module Resistor_SMD:R_0603_1608Metric (layer B.Cu)
-    (at 173.5075 91.52)
+    (at 171.4755 93.298)
     (descr "Resistor SMD 0603 (1608 Metric), square (rectangular) end terminal, IPC_7351 nominal, (Body size source: http://www.tortai-tech.com/upload/download/2011102023233369053.pdf), generated with kicad-footprint-generator")
     (tags resistor)
@@
   )
   (dimension 43 (width 0.12) (layer Dwgs.User)
-    (gr_text "43.000 mm" (at 128.9 61.441) (layer Dwgs.User)
+    (gr_text "43.000 mm" (at 128.9 62.441) (layer Dwgs.User)
       (effects (font (size 0.7 0.7) (thickness 0.15)))
     )
-    (feature1 (pts (xy 107.4 121.031) (xy 107.4 61.824579)))
-    (feature2 (pts (xy 150.4 121.031) (xy 150.4 61.824579)))
-    (crossbar (pts (xy 150.4 62.411) (xy 107.4 62.411)))
-    (arrow1a (pts (xy 107.4 62.411) (xy 108.526504 61.824579)))
-    (arrow1b (pts (xy 107.4 62.411) (xy 108.526504 62.997421)))
-    (arrow2a (pts (xy 150.4 62.411) (xy 149.273496 61.824579)))
-    (arrow2b (pts (xy 150.4 62.411) (xy 149.273496 62.997421)))
+    (feature1 (pts (xy 107.4 122.031) (xy 107.4 62.824579)))
+    (feature2 (pts (xy 150.4 122.031) (xy 150.4 62.824579)))
+    (crossbar (pts (xy 150.4 63.411) (xy 107.4 63.411)))
+    (arrow1a (pts (xy 107.4 63.411) (xy 108.526504 62.824579)))
+    (arrow1b (pts (xy 107.4 63.411) (xy 108.526504 63.997421)))
+    (arrow2a (pts (xy 150.4 63.411) (xy 149.273496 62.824579)))
+    (arrow2b (pts (xy 150.4 63.411) (xy 149.273496 63.997421)))
   )
   (gr_text TX (at 125.114 123.444 90) (layer F.SilkS)
@@
   (gr_line (start 180 80) (end 180 130) (layer Edge.Cuts) (width 0.05))
   (gr_line (start 120 80) (end 180 80) (layer Edge.Cuts) (width 0.05))
-  (segment (start 150.8 87.6) (end 150.8 89.992) (width 0.381) (layer F.Cu) (net 5))
-  (segment (start 148.9 91.892) (end 148.9 92.05) (width 0.381) (layer F.Cu) (net 5))
-  (segment (start 150.8 89.992) (end 148.9 91.892) (width 0.381) (layer F.Cu) (net 5))
-  (segment (start 150 87.6) (end 150 89.395) (width 0.381) (layer F.Cu) (net 6))
-  (segment (start 150 89.395) (end 149.225 90.17) (width 0.381) (layer F.Cu) (net 6))
-  (segment (start 149.225 90.17) (end 148.209 90.17) (width 0.381) (layer F.Cu) (net 6))
-  (segment (start 148.209 90.17) (end 146.939 91.44) (width 0.381) (layer F.Cu) (net 6))
-  (segment (start 147.989 93.95) (end 148.9 93.95) (width 0.381) (layer F.Cu) (net 6))
-  (segment (start 146.939 92.9) (end 147.989 93.95) (width 0.381) (layer F.Cu) (net 6))
-  (segment (start 146.939 91.44) (end 146.939 92.9) (width 0.381) (layer F.Cu) (net 6))
   (segment (start 140 104.578) (end 140.278 104.578) (width 0.2032) (layer B.Cu) (net 9))
   (segment (start 142.686 102.17) (end 144.325 102.17) (width 0.2032) (layer B.Cu) (net 9))
