File: argon-children/benzene-16/benzene-16.sch (KiCad schematic (older format))
At the start: 17 parts, among them U1 Conn1, U2 SPI FLASH, U3 Conn2, U4 LMC555, U5 IS25WP256D-xM

Commit message: Argon USB & custom footprint for DIP-16
Parts:
- U5: footprint Package_DIP:DIP-16_W7.62mm_Socket -> benzene:DIP-16_W15.24mm
Changed lines of the file:
@@
 F 0 "U5" H 8200 3681 50  0000 C CNN
 F 1 "IS25WP256D-xM" H 8200 3590 50  0000 C CNN
-F 2 "Package_DIP:DIP-16_W7.62mm_Socket" H 8250 3600 50  0001 C CNN
+F 2 "benzene:DIP-16_W15.24mm" H 8250 3600 50  0001 C CNN
 F 3 "http://www.issi.com/WW/pdf/IS25LP(WP)256D.pdf" H 8250 2500 50  0001 C CNN
 	1    8200 3000

Commit message: Argon PCB - part 2 + logo
Parts:
- C4: value 1uF -> 100nF
- R7: value 100K -> 1M
Changed lines of the file:
@@
 P 6550 5850
 F 0 "R7" V 6500 6050 50  0000 C CNN
-F 1 "100K" V 6500 5500 50  0000 L CNN
+F 1 "1M" V 6500 5500 50  0000 L CNN
 F 2 "Resistor_SMD:R_0603_1608Metric" V 6480 5850 50  0001 C CNN
 F 3 "~" H 6550 5850 50  0001 C CNN
@@
 P 7600 5850
 F 0 "C4" V 7650 6000 50  0000 C CNN
-F 1 "1uF" V 7650 5650 50  0000 C CNN
+F 1 "100nF" V 7650 5650 50  0000 C CNN
 F 2 "Capacitor_SMD:C_0603_1608Metric" H 7600 5850 50  0001 C CNN
 F 3 "~" H 7600 5850 50  0001 C CNN

Commit message: Benzene schematic
Parts:
- removed C1: 100nF, Capacitor_SMD:C_0603_1608Metric, symbol Device:C
- removed C2: 10uF, Capacitor_SMD:C_0603_1608Metric, symbol Device:C
- removed R1, R2, R3, R4: 47R, Resistor_SMD:R_0603_1608Metric, symbol Device:R
- removed U1: Conn1, Connector_PinHeader_2.54mm:PinHeader_1x02_P2.54mm_Vertical, symbol ArgonComponents:Conn1
- removed U2: SPI FLASH, benzene:DIP-8_W7.62mm_Socket, symbol ArgonComponents:SPI_FLASH
- removed U3: Conn2, Connector_PinHeader_2.54mm:PinHeader_1x04_P2.54mm_Vertical, symbol ArgonComponents:Conn2
- removed U5: IS25WP256D-xM, benzene:DIP-16_W15.24mm, symbol Memory_Flash:IS25WP256D-xM
- added C?: 100nF, Capacitor_SMD:C_0603_1608Metric, symbol Device:C
- added C?: 10uF, Capacitor_SMD:C_0603_1608Metric, symbol Device:C
- added R? (x4): 47R, Resistor_SMD:R_0603_1608Metric, symbol Device:R
- added U?: DIP-8, Package_SO:SOIC-8_5.23x5.23mm_P1.27mm, symbol ArgonComponents:spi_flash_dip_8
- added U?: DIP-16, Package_SO:SOIC-16W_7.5x10.3mm_P1.27mm, symbol ArgonComponents:spi_flash_dip_16
- added U?: Conn1, Connector_PinHeader_2.54mm:PinHeader_1x02_P2.54mm_Vertical, symbol ArgonComponents:Conn1
- added U?: Conn2, Connector_PinHeader_2.54mm:PinHeader_1x04_P2.54mm_Vertical, symbol ArgonComponents:Conn2
Connections:
- net GND: now also C3.1, C?.2, C?.2, U?.2 (GND), U?.4 (GND); no longer C3.2
- net V3V3: now also R5.1, C?.1, C?.1, U?.1 (V3V3), U?.3 (~WP), U?.7 (~RESET), U?.8 (VCC); no longer R5.2
- net at U4.5 (CV): now also C3.2; no longer C3.1
- net ~CS: no longer names the net of U4.2 (TR)
- net ~CS: no longer R5.1
- new net: R?.1, U?.1 (~CS)
- new net: R?.1, U?.2 (MISO)
- new net: R?.1, U?.5 (MOSI)
- new net: R?.1, U?.6 (CLK)
- new net CS: R5.2, R?.2, U?.4 (CS)
- new net MISO: R?.2, U?.3 (MISO)
- new net MOSI: R?.2, U?.2 (MOSI)
- new net SCK: R?.2, U?.1 (SCK)
Other:
- moved on the sheet: C3, C4, D1, R5, R6, R7, U4

Commit message: Benzene schematic
Parts:
- added R? (x4): 47R, Resistor_SMD:R_0603_1608Metric, symbol Device:R
- C3: value 10uF -> 10nF
- C4: symbol Device:CP1 -> Device:C
- C?: symbol Device:C -> Device:CP1
Connections:
- net CS: now also R?.2
- net GND: now also U?.10 (GND)
- net MISO: now also R?.2
- net MOSI: now also R?.2
- net SCK: now also R?.2
- net V3V3: now also U?.2 (VCC), U?.3 (~RESET), U?.9 (~WP)
- net at U?.15 (MOSI): now also R?.1
- net at U?.16 (SCK): now also R?.1
- net at U?.7 (~CS): now also R?.1
- net at U?.8 (MISO): now also R?.1
- no-connect marks 0 -> 1
Other:
- moved on the sheet: U?
Changed lines of the file:
@@
 $EndComp
 $Comp
-L Device:CP1 C4
+L Device:C C4
 U 1 1 5FD76E93
 P 7600 5750
@@
 P 4550 5250
 F 0 "C3" V 4500 5150 50  0000 C CNN
-F 1 "10uF" V 4600 5100 50  0000 C CNN
+F 1 "10nF" V 4600 5100 50  0000 C CNN
 F 2 "Capacitor_SMD:C_0603_1608Metric" H 4588 5100 50  0001 C CNN
 F 3 "~" H 4550 5250 50  0001 C CNN
@@
 Wire Wire Line
 	8000 5050 8000 5200
-$Comp
-L Device:C C?
-U 1 1 5FE70F3F
-P 5750 3150
-F 0 "C?" V 5800 3250 50  0000 C CNN
-F 1 "100nF" V 5700 3200 50  0000 L CNN
-F 2 "Capacitor_SMD:C_0603_1608Metric" H 5788 3000 50  0001 C CNN
-F 3 "~" H 5750 3150 50  0001 C CNN
-	1    5750 3150
-	0    1    -1   0
-$EndComp
 Wire Wire Line
 	5900 3150 6050 3150
 Wire Wire Line
 	5600 3150 5450 3150
-$Comp
-L Device:C C?
-U 1 1 5FE70F47
-P 5750 2850
-F 0 "C?" V 5800 2950 50  0000 C CNN
-F 1 "10uF" V 5700 3000 50  0000 C CNN
-F 2 "Capacitor_SMD:C_0603_1608Metric" H 5788 2700 50  0001 C CNN
-F 3 "~" H 5750 2850 50  0001 C CNN
-	1    5750 2850
-	0    1    -1   0
-$EndComp
 Wire Wire Line
 	5900 2850 6050 2850
@@
 L ArgonComponents:spi_flash_dip_16 U?
 U 1 1 5FE66CFF
-P 7850 3050
-F 0 "U?" H 7500 3500 50  0000 C CNN
-F 1 "DIP-16" H 8100 2600 50  0000 C CNN
-F 2 "Package_SO:SOIC-16W_7.5x10.3mm_P1.27mm" H 7900 3650 50  0001 C CNN
-F 3 "http://www.issi.com/WW/pdf/IS25LP(WP)256D.pdf" H 7900 2550 50  0001 C CNN
-	1    7850 3050
+P 8500 2900
+F 0 "U?" H 8150 3350 50  0000 C CNN
+F 1 "DIP-16" H 8750 2450 50  0000 C CNN
+F 2 "Package_SO:SOIC-16W_7.5x10.3mm_P1.27mm" H 8550 3500 50  0001 C CNN
+F 3 "http://www.issi.com/WW/pdf/IS25LP(WP)256D.pdf" H 8550 2400 50  0001 C CNN
+	1    8500 2900
 	1    0    0    -1
 $EndComp
@@
 Wire Wire Line
 	2150 1950 2150 2350
+$Comp
+L Device:R R?
+U 1 1 5FE49267
+P 9450 2350
+F 0 "R?" H 9350 2300 50  0000 C CNN
+F 1 "47R" H 9250 2400 50  0000 L CNN
+F 2 "Resistor_SMD:R_0603_1608Metric" V 9380 2350 50  0001 C CNN
+F 3 "~" H 9450 2350 50  0001 C CNN
+	1    9450 2350
+	-1   0    0    1
+$EndComp
+$Comp
+L Device:R R?
+U 1 1 5FE49BCE
+P 7800 2350
+F 0 "R?" H 7700 2300 50  0000 C CNN
+F 1 "47R" H 7600 2400 50  0000 L CNN
+F 2 "Resistor_SMD:R_0603_1608Metric" V 7730 2350 50  0001 C CNN
+F 3 "~" H 7800 2350 50  0001 C CNN
+	1    7800 2350
+	-1   0    0    1
+$EndComp
+NoConn ~ 8000 3100
+$Comp
+L power:GND #PWR?
+U 1 1 5FE4C677
+P 8500 3600
+F 0 "#PWR?" H 8500 3350 50  0001 C CNN
+F 1 "GND" V 8505 3472 50  0000 R CNN
+F 2 "" H 8500 3600 50  0001 C CNN
+F 3 "" H 8500 3600 50  0001 C CNN
+	1    8500 3600
+	1    0    0    -1
+$EndComp
+Wire Wire Line
+	8500 3400 8500 3600
+Wire Wire Line
+	9000 3000 9350 3000
+Wire Wire Line
+	7650 3000 8000 3000
+Text GLabel 7650 3000 0    50   Input ~ 0
+V3V3
+Text GLabel 9350 3000 2    50   Input ~ 0
+V3V3
+Wire Wire Line
+	9000 2700 9450 2700
+Wire Wire Line
+	9450 2700 9450 2500
+Wire Wire Line
+	8500 2250 8500 2400
+Wire Wire Line
+	8550 2250 8500 2250
+Text GLabel 8550 2250 2    50   Input ~ 0
+V3V3
+$Comp
+L Device:R R?
+U 1 1 5FE66E01
+P 7500 2350
+F 0 "R?" H 7400 2300 50  0000 C CNN
+F 1 "47R" H 7300 2400 50  0000 L CNN
+F 2 "Resistor_SMD:R_0603_1608Metric" V 7430 2350 50  0001 C CNN
+F 3 "~" H 7500 2350 50  0001 C CNN
+	1    7500 2350
+	-1   0    0    1
+$EndComp
+$Comp
+L Device:R R?
+U 1 1 5FE6703E
+P 7200 2350
+F 0 "R?" H 7100 2300 50  0000 C CNN
+F 1 "47R" H 7000 2400 50  0000 L CNN
+F 2 "Resistor_SMD:R_0603_1608Metric" V 7130 2350 50  0001 C CNN
+F 3 "~" H 7200 2350 50  0001 C CNN
+	1    7200 2350
+	-1   0    0    1
+$EndComp
+Wire Wire Line
+	8000 2900 7200 2900
+Wire Wire Line
+	7200 2900 7200 2500
+Wire Wire Line
+	7500 2500 7500 2800
+Wire Wire Line
+	7500 2800 8000 2800
+Wire Wire Line
+	8000 2700 7800 2700
+Wire Wire Line
+	7800 2700 7800 2500
+$Comp
+L Device:C C?
+U 1 1 5FE70F3F
+P 5750 3150
+F 0 "C?" V 5800 3000 50  0000 C CNN
+F 1 "100nF" V 5700 2850 50  0000 L CNN
+F 2 "Capacitor_SMD:C_0603_1608Metric" H 5788 3000 50  0001 C CNN
+F 3 "~" H 5750 3150 50  0001 C CNN
+	1    5750 3150
+	0    1    -1   0
+$EndComp
+$Comp
+L Device:CP1 C?
+U 1 1 5FE70F47
+P 5750 2850
+F 0 "C?" V 5800 2700 50  0000 C CNN
+F 1 "10uF" V 5700 2700 50  0000 C CNN
+F 2 "Capacitor_SMD:C_0603_1608Metric" H 5788 2700 50  0001 C CNN
+F 3 "~" H 5750 2850 50  0001 C CNN
+	1    5750 2850
+	0    1    -1   0
+$EndComp
+Text GLabel 8200 1850 1    50   Input ~ 0
+CS
+Text GLabel 8800 1850 1    50   Input ~ 0
+MISO
+Text GLabel 8600 1850 1    50   Input ~ 0
+MOSI
+Text GLabel 8400 1850 1    50   Input ~ 0
+SCK
+Wire Wire Line
+	8800 1850 8800 1950
+Wire Wire Line
+	8800 1950 9450 1950
+Wire Wire Line
+	9450 1950 9450 2200
+Wire Wire Line
+	7800 2200 7800 2100
+Wire Wire Line
+	7800 2100 8600 2100
+Wire Wire Line
+	8600 2100 8600 1850
+Wire Wire Line
+	8400 1850 8400 2000
+Wire Wire Line
+	8400 2000 7500 2000
+Wire Wire Line
+	7500 2000 7500 2200
+Wire Wire Line
+	7200 1900 8200 1900
+Wire Wire Line
+	8200 1900 8200 1850
+Wire Wire Line
+	7200 1900 7200 2200
 $EndSCHEMATC

Commit message: Benzene schematic - final
Parts:
- removed C?: 100nF, Capacitor_SMD:C_0603_1608Metric, symbol Device:C
- removed C?: 10uF, Capacitor_SMD:C_0603_1608Metric, symbol Device:CP1
- removed R? (x7): 47R, Resistor_SMD:R_0603_1608Metric, symbol Device:R
- added C1, C5: 10uF, Capacitor_SMD:C_0603_1608Metric, symbol Device:CP1
- added C2, C6: 100nF, Capacitor_SMD:C_0603_1608Metric, symbol Device:C
- added R3, R4, R5: 47R, Resistor_SMD:R_0603_1608Metric, symbol Device:R
- gave numbers to parts that had none: 5
- renumbered R5 to R1, R7 to R6, R6 to R7
Connections:
- net CS: now also R2.1, U1.1 (~CS), U5.7 (~CS); no longer R2.2, U2.4 (CS)
- net GND: now also C1.2, C2.1, C5.2, C6.1
- net MISO: now also U1.2 (MISO), U5.8 (MISO), R3.1; no longer U2.3 (MISO)
- net MOSI: now also U1.5 (MOSI), U5.15 (MOSI), R4.1; no longer U2.2 (MOSI)
- net SCK: now also U1.6 (CLK), U5.16 (SCK), R5.1; no longer U2.1 (SCK)
- net V3V3: now also C1.1, C2.2, C5.1, C6.2
- new net: R2.2, U2.4 (CS)
- new net: R3.2, U2.3 (MISO)
- new net: R4.2, U2.2 (MOSI)
- new net: R5.2, U2.1 (SCK)
Other:
- moved on the sheet: R2, U2, U3

Commit message: Benzene pcb
Parts:
- C1, C5: footprint Capacitor_SMD:C_0603_1608Metric -> Capacitor_Tantalum_SMD:CP_EIA-3216-18_Kemet-A
- U1: footprint Package_SO:SOIC-8_5.23x5.23mm_P1.27mm -> benzene:DIP-8_W7.62mm_Socket
- U3: renamed from U5; footprint Package_SO:SOIC-16W_7.5x10.3mm_P1.27mm -> benzene:DIP-16_W15.24mm
- renumbered U2 to J1, U3 to J2, U4 to U2
Changed lines of the file:
@@
 	5850 5650 5850 5900
 $Comp
-L Timer:LMC555xM U4
+L Timer:LMC555xM U2
 U 1 1 5FD3E29C
 P 5850 5250
-F 0 "U4" H 5550 5600 50  0000 C CNN
+F 0 "U2" H 5550 5600 50  0000 C CNN
 F 1 "LMC555" H 6050 5600 50  0000 C CNN
 F 2 "Package_SO:VSSOP-8_3.0x3.0mm_P0.65mm" H 6700 4850 50  0001 C CNN
@@
 	8000 5050 8000 5200
 $Comp
-L ArgonComponents:spi_flash_dip_16 U5
+L ArgonComponents:spi_flash_dip_16 U3
 U 1 1 5FE66CFF
 P 8500 2900
-F 0 "U5" H 8150 3350 50  0000 C CNN
+F 0 "U3" H 8150 3350 50  0000 C CNN
 F 1 "DIP-16" H 8750 2450 50  0000 C CNN
-F 2 "Package_SO:SOIC-16W_7.5x10.3mm_P1.27mm" H 8550 3500 50  0001 C CNN
+F 2 "benzene:DIP-16_W15.24mm" H 8550 3500 50  0001 C CNN
 F 3 "http://www.issi.com/WW/pdf/IS25LP(WP)256D.pdf" H 8550 2400 50  0001 C CNN
 	1    8500 2900
@@
 $EndComp
 $Comp
-L ArgonComponents:Conn1 U3
+L ArgonComponents:Conn1 J2
 U 1 1 5FE8D895
 P 5650 2850
-F 0 "U3" V 5850 2850 50  0000 L CNN
+F 0 "J2" V 5850 2850 50  0000 L CNN
 F 1 "Conn1" V 5662 3038 50  0001 L CNN
 F 2 "Connector_PinHeader_2.54mm:PinHeader_1x02_P2.54mm_Vertical" H 5550 3150 50  0001 C CNN
@@
 $EndComp
 $Comp
-L ArgonComponents:Conn2 U2
+L ArgonComponents:Conn2 J1
 U 1 1 5FF5C69A
 P 5100 1500
-F 0 "U2" H 5150 1800 50  0000 R CNN
+F 0 "J1" H 5150 1800 50  0000 R CNN
 F 1 "Conn2" V 5050 1100 50  0001 R CNN
 F 2 "Connector_PinHeader_2.54mm:PinHeader_1x04_P2.54mm_Vertical" H 5000 1800 50  0001 C CNN
@@
 F 0 "C5" V 8850 1900 50  0000 C CNN
 F 1 "10uF" V 8850 1500 50  0000 C CNN
-F 2 "Capacitor_SMD:C_0603_1608Metric" H 8938 1550 50  0001 C CNN
+F 2 "Capacitor_Tantalum_SMD:CP_EIA-3216-18_Kemet-A" H 8938 1550 50  0001 C CNN
 F 3 "~" H 8900 1700 50  0001 C CNN
 	1    8900 1700
@@
 F 0 "U1" H 2900 3300 50  0000 C CNN
 F 1 "DIP-8" H 3550 2600 50  0000 C CNN
-F 2 "Package_SO:SOIC-8_5.23x5.23mm_P1.27mm" H 3250 2950 50  0001 C CNN
+F 2 "benzene:DIP-8_W7.62mm_Socket" H 3250 2950 50  0001 C CNN
 F 3 "http://www.winbond.com/resource-files/w25q32jv%20revg%2003272018%20plus.pdf" H 3250 2950 50  0001 C CNN
 	1    3250 2950
@@
 F 0 "C1" V 3600 2050 50  0000 C CNN
 F 1 "10uF" V 3600 1650 50  0000 C CNN
-F 2 "Capacitor_SMD:C_0603_1608Metric" H 3688 1700 50  0001 C CNN
+F 2 "Capacitor_Tantalum_SMD:CP_EIA-3216-18_Kemet-A" H 3688 1700 50  0001 C CNN
 F 3 "~" H 3650 1850 50  0001 C CNN
 	1    3650 1850

Commit message: Benzene PCB
Parts:
- C1, C5: footprint Capacitor_Tantalum_SMD:CP_EIA-3216-18_Kemet-A -> argon:CP_EIA-3216-18_Kemet-A
- U1: footprint benzene:DIP-8_W7.62mm_Socket -> benzene:DIP-8_W7.62mm_Socket_wihtout_lines
- U3: footprint benzene:DIP-16_W15.24mm -> benzene:DIP-16_W15.24mm_without_lines
Connections:
- net CS: now also U2.2 (TR)
- net V3V3: now also U3.1 (~HOLD)
- no-connect marks 1 -> 0
Changed lines of the file:
@@
 Wire Wire Line
 	5850 5650 5850 5900
-$Comp
-L Timer:LMC555xM U2
-U 1 1 5FD3E29C
-P 5850 5250
-F 0 "U2" H 5550 5600 50  0000 C CNN
-F 1 "LMC555" H 6050 5600 50  0000 C CNN
-F 2 "Package_SO:VSSOP-8_3.0x3.0mm_P0.65mm" H 6700 4850 50  0001 C CNN
-F 3 "http://www.ti.com/lit/ds/symlink/lmc555.pdf" H 6700 4850 50  0001 C CNN
-	1    5850 5250
-	1    0    0    -1
-$EndComp
 Connection ~ 7250 5750
 Wire Wire Line
@@
 $EndComp
 Wire Wire Line
-	5300 5050 5000 5050
-Wire Wire Line
 	5000 4700 4700 4700
 Wire Wire Line
@@
 F 0 "U3" H 8150 3350 50  0000 C CNN
 F 1 "DIP-16" H 8750 2450 50  0000 C CNN
-F 2 "benzene:DIP-16_W15.24mm" H 8550 3500 50  0001 C CNN
+F 2 "benzene:DIP-16_W15.24mm_without_lines" H 8550 3500 50  0001 C CNN
 F 3 "http://www.issi.com/WW/pdf/IS25LP(WP)256D.pdf" H 8550 2400 50  0001 C CNN
 	1    8500 2900
@@
 Text GLabel 2350 3050 0    50   Input ~ 0
 SCK
-NoConn ~ 8000 3100
 $Comp
 L power:GND #PWR08
@@
 	6300 2000 6300 1750
 Wire Wire Line
-	7650 3000 8000 3000
+	7750 3000 8000 3000
 Text GLabel 7600 3100 0    50   Input ~ 0
 V3V3
 Wire Wire Line
-	7600 3100 7650 3100
-Wire Wire Line
-	7650 3100 7650 3000
+	7600 3100 7750 3100
+Wire Wire Line
+	7750 3100 7750 3000
 Text GLabel 7600 2500 0    50   Input ~ 0
 MOSI
@@
 F 0 "C5" V 8850 1900 50  0000 C CNN
 F 1 "10uF" V 8850 1500 50  0000 C CNN
-F 2 "Capacitor_Tantalum_SMD:CP_EIA-3216-18_Kemet-A" H 8938 1550 50  0001 C CNN
+F 2 "argon:CP_EIA-3216-18_Kemet-A" H 8938 1550 50  0001 C CNN
 F 3 "~" H 8900 1700 50  0001 C CNN
 	1    8900 1700
@@
 F 0 "U1" H 2900 3300 50  0000 C CNN
 F 1 "DIP-8" H 3550 2600 50  0000 C CNN
-F 2 "benzene:DIP-8_W7.62mm_Socket" H 3250 2950 50  0001 C CNN
+F 2 "benzene:DIP-8_W7.62mm_Socket_wihtout_lines" H 3250 2950 50  0001 C CNN
 F 3 "http://www.winbond.com/resource-files/w25q32jv%20revg%2003272018%20plus.pdf" H 3250 2950 50  0001 C CNN
 	1    3250 2950
@@
 F 0 "C1" V 3600 2050 50  0000 C CNN
 F 1 "10uF" V 3600 1650 50  0000 C CNN
-F 2 "Capacitor_Tantalum_SMD:CP_EIA-3216-18_Kemet-A" H 3688 1700 50  0001 C CNN
+F 2 "argon:CP_EIA-3216-18_Kemet-A" H 3688 1700 50  0001 C CNN
 F 3 "~" H 3650 1850 50  0001 C CNN
 	1    3650 1850
@@
 Wire Wire Line
 	6100 2850 6100 2950
+Wire Wire Line
+	8000 3100 7750 3100
+Connection ~ 7750 3100
+Wire Wire Line
+	5000 5050 5350 5050
+$Comp
+L Timer:LMC555xM U2
+U 1 1 5FD3E29C
+P 5850 5250
+F 0 "U2" H 5550 5600 50  0000 C CNN
+F 1 "LMC555" H 6050 5600 50  0000 C CNN
+F 2 "Package_SO:VSSOP-8_3.0x3.0mm_P0.65mm" H 6700 4850 50  0001 C CNN
+F 3 "http://www.ti.com/lit/ds/symlink/lmc555.pdf" H 6700 4850 50  0001 C CNN
+	1    5850 5250
+	1    0    0    -1
+$EndComp
 $EndSCHEMATC
