File: argon-children/benzene-16/benzene-16.kicad_pcb (KiCad board)
At the start: 2 copper layers, 25 x 30 mm, 20 parts, among them J1 Conn2, J2 Conn1, U1 DIP-8, U2 LMC555, U3 DIP-16

Commit message: Final touches
Routing:
- net V3V3: track 80.6 -> 78.5 mm, vias 4 -> 3
Changed lines of the file:
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@@
     (thickness 1.6)
     (drawings 13)
-    (tracks 183)
+    (tracks 180)
     (zones 0)
     (modules 20)
@@
   )
   (layers
-    (0 F.Cu signal)
+    (0 F.Cu signal hide)
     (31 B.Cu signal)
     (32 B.Adhes user hide)
@@
   (segment (start 97.201 52.1715) (end 97.351 52.1715) (width 0.381) (layer B.Cu) (net 1))
   (segment (start 97.201 52.1715) (end 97.113 52.1715) (width 0.2032) (layer B.Cu) (net 1))
-  (segment (start 97.113 52.1715) (end 95.953 53.3315) (width 0.2032) (layer B.Cu) (net 1))
-  (segment (start 95.953 58.061) (end 97.201 59.309) (width 0.2032) (layer B.Cu) (net 1))
-  (segment (start 95.953 53.3315) (end 95.953 58.061) (width 0.2032) (layer B.Cu) (net 1))
   (segment (start 103.94892 59.87454) (end 102.63828 58.5639) (width 0.2032) (layer F.Cu) (net 1))
   (segment (start 102.63828 58.5639) (end 98.7978 58.5639) (width 0.2032) (layer F.Cu) (net 1))
@@
   (segment (start 110.304 56.062) (end 110.304 55.9985) (width 0.2032) (layer F.Cu) (net 1))
   (segment (start 106.4356 52.2647) (end 106.4356 51.8761) (width 0.2032) (layer B.Cu) (net 1))
-  (segment (start 106.4356 51.8761) (end 105.351 50.7915) (width 0.2032) (layer B.Cu) (net 1))
-  (segment (start 98.581 50.7915) (end 97.201 52.1715) (width 0.2032) (layer B.Cu) (net 1))
-  (segment (start 105.351 50.7915) (end 98.581 50.7915) (width 0.2032) (layer B.Cu) (net 1))
-  (segment (start 105.7925 69.5465) (end 110.1515 73.9055) (width 0.2032) (layer B.Cu) (net 1))
+  (segment (start 106.4356 51.8761) (end 105.351 50.7915) (width 0.381) (layer B.Cu) (net 1))
+  (segment (start 98.581 50.7915) (end 97.201 52.1715) (width 0.381) (layer B.Cu) (net 1))
+  (segment (start 105.351 50.7915) (end 98.581 50.7915) (width 0.381) (layer B.Cu) (net 1))
+  (segment (start 105.7925 69.5465) (end 110.1515 73.9055) (width 0.381) (layer B.Cu) (net 1))
   (segment (start 105.571 69.5465) (end 105.7925 69.5465) (width 0.2032) (layer B.Cu) (net 1))
   (segment (start 112.192 63.085) (end 111.485 63.085) (width 0.381) (layer B.Cu) (net 1))
@@
   (segment (start 107.8625 62.285) (end 106.367 63.7805) (width 0.381) (layer B.Cu) (net 1))
   (segment (start 110.685 62.285) (end 107.8625 62.285) (width 0.381) (layer B.Cu) (net 1))
+  (segment (start 96.526 52.1715) (end 95.953 52.7445) (width 0.381) (layer B.Cu) (net 1))
+  (segment (start 97.201 52.1715) (end 96.526 52.1715) (width 0.381) (layer B.Cu) (net 1))
+  (segment (start 95.953 58.061) (end 97.201 59.309) (width 0.381) (layer B.Cu) (net 1))
+  (segment (start 95.953 52.7445) (end 95.953 58.061) (width 0.381) (layer B.Cu) (net 1))
   (segment (start 109.14576 52.25454) (end 109.1356 52.2647) (width 0.381) (layer B.Cu) (net 2))
   (segment (start 111.56892 52.25454) (end 109.14576 52.25454) (width 0.381) (layer B.Cu) (net 2))
@@
   (segment (start 110.9645 70.54) (end 109.971 69.5465) (width 0.381) (layer B.Cu) (net 2))
   (segment (start 112.463 70.54) (end 110.9645 70.54) (width 0.381) (layer B.Cu) (net 2))
-  (segment (start 112.463 70.8575) (end 112.463 70.54) (width 0.381) (layer F.Cu) (net 2))
-  (via (at 114.876 71.8735) (size 0.8) (drill 0.4) (layers F.Cu B.Cu) (net 2))
-  (segment (start 114.876 71.8735) (end 113.479 71.8735) (width 0.381) (layer F.Cu) (net 2))
-  (segment (start 113.479 71.8735) (end 112.463 70.8575) (width 0.381) (layer F.Cu) (net 2))
-  (segment (start 115.381 71.302) (end 115.381 70.0315) (width 0.381) (layer B.Cu) (net 2))
-  (segment (start 114.876 71.8735) (end 115.381 71.302) (width 0.381) (layer B.Cu) (net 2))
   (segment (start 107.263 65.9045) (end 105.571 67.5965) (width 0.381) (layer B.Cu) (net 2))
   (segment (start 108.111 65.9045) (end 107.263 65.9045) (width 0.381) (layer B.Cu) (net 2))
@@
   (segment (start 101.922 70.8575) (end 101.922 67.492) (width 0.381) (layer F.Cu) (net 2))
   (segment (start 101.922 67.492) (end 103.446 65.968) (width 0.381) (layer F.Cu) (net 2))
+  (segment (start 114.8725 70.54) (end 115.381 70.0315) (width 0.381) (layer F.Cu) (net 2))
+  (segment (start 112.463 70.54) (end 114.8725 70.54) (width 0.381) (layer F.Cu) (net 2))
   (segment (start 112.971 68.8255) (end 113.479 69.3335) (width 0.2032) (layer B.Cu) (net 3))
   (segment (start 112.463 68.8255) (end 112.971 68.8255) (width 0.2032) (layer B.Cu) (net 3))
